Commit message: Updated URDF on robotic_arm so it rotates on the right axis

File: URDF/robotic_arm.urdf (robot description, URDF)
Before this commit: robot robot_arm, 12 links, 11 joints
Links:
- added link Elbow_link_top; visual box size=0.2 0.2 0.2
- added link Wrist_link_top; visual box size=0.2 0.2 0.2
- link Wrist1_link: geometry visual cylinder length=0.15 radius=0.1
- link Wrist1_link_j: geometry visual box size=0.2 0.2 0.2
- link Wrist2_link: geometry visual cylinder length=0.15 radius=0.1
- link Wrist_link_j: geometry visual box size=0.2 0.2 0.2
Joints:
- added joint Elbow_top_fixed: type fixed, parent Elbow_link, child Elbow_link_top
- added joint Wrist_top_fixed: type fixed, parent Wrist_link, child Wrist_link_top
- joint Elbow_to_wrist: origin xyz=0.0 -0.1 0.7 rpy=0 0 0 -> xyz=0.7 -0.2 0.0 rpy=0 0 0
- joint Wris2_to_wrist3: axis 1 0 0 -> 0 1 0; origin xyz=-0.5 0.0 0.0 rpy=0 0 0 -> xyz=0.0 0.34 0.0 rpy=0 0 0
- joint Wrist1_to_wrist2: origin xyz=0.0 0.1 0.5 rpy=0 0 0 -> xyz=0.0 0.0 -0.34 rpy=0 0 0
- joint Wrist_to_wrist1: origin xyz=0.0 0.0 0.7 rpy=0 0 0 -> xyz=0.7 0.2 0.0 rpy=0 0 0
